File: hardware/sunrise_alarmclock.brd (EAGLE design)
At the start: 48.6 x 45.4 mm, 26 parts, among them IC1 ATMEGA328P, IC2 WTV020, IC3 TinyRTC, IC4 HC-05, IC5 LD117AS33TR

Commit message: hardware: added components values
Parts:
- R1, R3, R5, R7: value (none) -> 18k
- R2, R4, R6, R8: value (none) -> 33k
Changed lines of the file:
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@@
 <attribute name="VALUE" x="24.126" y="32.385" size="1.27" layer="28" ratio="10" rot="MR270"/>
 </element>
-<element name="R1" library="rcl" package="M1206" value="" x="4.6275" y="29.52" smashed="yes">
+<element name="R1" library="rcl" package="M1206" value="18k" x="4.6275" y="29.52" smashed="yes">
 <attribute name="NAME" x="7.3575" y="28.79" size="1.27" layer="25"/>
 <attribute name="VALUE" x="3.3575" y="26.98" size="1.27" layer="27"/>
 </element>
-<element name="R2" library="rcl" package="M1206" value="" x="4.6275" y="32.48" smashed="yes">
+<element name="R2" library="rcl" package="M1206" value="33k" x="4.6275" y="32.48" smashed="yes">
 <attribute name="NAME" x="7.3575" y="31.75" size="1.27" layer="25"/>
 <attribute name="VALUE" x="3.3575" y="29.94" size="1.27" layer="27"/>
@@
 <attribute name="VALUE" x="41.85" y="8.9" size="1.016" layer="28" rot="MR0"/>
 </element>
-<element name="R3" library="rcl" package="M1206" value="" x="7.75" y="10.25" smashed="yes" rot="R90">
+<element name="R3" library="rcl" package="M1206" value="18k" x="7.75" y="10.25" smashed="yes" rot="R90">
 <attribute name="NAME" x="6.48" y="8.98" size="1.27" layer="25" rot="R90"/>
 <attribute name="VALUE" x="10.29" y="8.98" size="1.27" layer="27" rot="R90"/>
 </element>
-<element name="R5" library="rcl" package="M1206" value="" x="10.25" y="10.25" smashed="yes" rot="R90">
+<element name="R5" library="rcl" package="M1206" value="18k" x="10.25" y="10.25" smashed="yes" rot="R90">
 <attribute name="NAME" x="15.48" y="8.98" size="1.27" layer="25" rot="R90"/>
 <attribute name="VALUE" x="12.79" y="8.98" size="1.27" layer="27" rot="R90"/>
 </element>
-<element name="R7" library="rcl" package="M1206" value="" x="12.75" y="10.25" smashed="yes" rot="R90">
+<element name="R7" library="rcl" package="M1206" value="18k" x="12.75" y="10.25" smashed="yes" rot="R90">
 <attribute name="NAME" x="17.23" y="8.98" size="1.27" layer="25" rot="R90"/>
 <attribute name="VALUE" x="15.29" y="8.98" size="1.27" layer="27" rot="R90"/>
 </element>
-<element name="R4" library="rcl" package="M1206" value="" x="7.75" y="4.25" smashed="yes" rot="R90">
+<element name="R4" library="rcl" package="M1206" value="33k" x="7.75" y="4.25" smashed="yes" rot="R90">
 <attribute name="NAME" x="6.48" y="2.98" size="1.27" layer="25" rot="R90"/>
 <attribute name="VALUE" x="10.29" y="2.98" size="1.27" layer="27" rot="R90"/>
 </element>
-<element name="R6" library="rcl" package="M1206" value="" x="10.25" y="4.25" smashed="yes" rot="R90">
+<element name="R6" library="rcl" package="M1206" value="33k" x="10.25" y="4.25" smashed="yes" rot="R90">
 <attribute name="NAME" x="15.48" y="2.98" size="1.27" layer="25" rot="R90"/>
 <attribute name="VALUE" x="12.79" y="2.98" size="1.27" layer="27" rot="R90"/>
 </element>
-<element name="R8" library="rcl" package="M1206" value="" x="12.75" y="4.25" smashed="yes" rot="R90">
+<element name="R8" library="rcl" package="M1206" value="33k" x="12.75" y="4.25" smashed="yes" rot="R90">
 <attribute name="NAME" x="17.23" y="2.98" size="1.27" layer="25" rot="R90"/>
 <attribute name="VALUE" x="15.29" y="2.98" size="1.27" layer="27" rot="R90"/>

Commit message: hardware: fixed values of resistor towards the voice module. added note about connection of photo resistor to pin PC1
Parts:
- R3, R5, R7: value 18k -> 100R
- R4, R6, R8: value 33k -> NA
Connections:
- new net N$22: IC1.24
Changed lines of the file:
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@@
 <attribute name="VALUE" x="41.85" y="8.9" size="1.016" layer="28" rot="MR0"/>
 </element>
-<element name="R3" library="rcl" package="M1206" value="18k" x="7.75" y="10.25" smashed="yes" rot="R90">
+<element name="R3" library="rcl" package="M1206" value="100R" x="7.75" y="10.25" smashed="yes" rot="R90">
 <attribute name="NAME" x="6.48" y="8.98" size="1.27" layer="25" rot="R90"/>
 <attribute name="VALUE" x="10.29" y="8.98" size="1.27" layer="27" rot="R90"/>
 </element>
-<element name="R5" library="rcl" package="M1206" value="18k" x="10.25" y="10.25" smashed="yes" rot="R90">
+<element name="R5" library="rcl" package="M1206" value="100R" x="10.25" y="10.25" smashed="yes" rot="R90">
 <attribute name="NAME" x="15.48" y="8.98" size="1.27" layer="25" rot="R90"/>
 <attribute name="VALUE" x="12.79" y="8.98" size="1.27" layer="27" rot="R90"/>
 </element>
-<element name="R7" library="rcl" package="M1206" value="18k" x="12.75" y="10.25" smashed="yes" rot="R90">
+<element name="R7" library="rcl" package="M1206" value="100R" x="12.75" y="10.25" smashed="yes" rot="R90">
 <attribute name="NAME" x="17.23" y="8.98" size="1.27" layer="25" rot="R90"/>
 <attribute name="VALUE" x="15.29" y="8.98" size="1.27" layer="27" rot="R90"/>
 </element>
-<element name="R4" library="rcl" package="M1206" value="33k" x="7.75" y="4.25" smashed="yes" rot="R90">
+<element name="R4" library="rcl" package="M1206" value="NA" x="7.75" y="4.25" smashed="yes" rot="R90">
 <attribute name="NAME" x="6.48" y="2.98" size="1.27" layer="25" rot="R90"/>
 <attribute name="VALUE" x="10.29" y="2.98" size="1.27" layer="27" rot="R90"/>
 </element>
-<element name="R6" library="rcl" package="M1206" value="33k" x="10.25" y="4.25" smashed="yes" rot="R90">
+<element name="R6" library="rcl" package="M1206" value="NA" x="10.25" y="4.25" smashed="yes" rot="R90">
 <attribute name="NAME" x="15.48" y="2.98" size="1.27" layer="25" rot="R90"/>
 <attribute name="VALUE" x="12.79" y="2.98" size="1.27" layer="27" rot="R90"/>
 </element>
-<element name="R8" library="rcl" package="M1206" value="33k" x="12.75" y="4.25" smashed="yes" rot="R90">
+<element name="R8" library="rcl" package="M1206" value="NA" x="12.75" y="4.25" smashed="yes" rot="R90">
 <attribute name="NAME" x="17.23" y="2.98" size="1.27" layer="25" rot="R90"/>
 <attribute name="VALUE" x="15.29" y="2.98" size="1.27" layer="27" rot="R90"/>
@@
 <wire x1="3.366" y1="23.404" x2="3.25" y2="23.52" width="0.4064" layer="1"/>
 </signal>
+<signal name="N$22">
+<contactref element="IC1" pad="24"/>
+</signal>
 </signals>
